Commit message: update two_scara_collaboration

File: urdf/blue_cylinder.urdf (robot description, URDF)
Before this commit: robot blue_cylinder, 1 links, 0 joints
Links:
- link base_link: mass 0.00001 -> 0.006; geometry collision sphere radius=0.02; visual sphere radius=0.02

File: urdf/conveyor_belt.urdf (robot description, URDF)
Before this commit: robot conveyor_belt, 2 links, 1 joints
Links:
- added link railing1, mass 1.0; collision box size=3 0.01 0.1; visual box size=3 0.01 0.1
- added link railing2, mass 1.0; collision box size=3 0.01 0.1; visual box size=3 0.01 0.1
- added link railing3, mass 1.0; collision box size=3 0.01 0.025; visual box size=3 0.01 0.025
- link base_link: mass 1 -> 1.0; geometry collision box size=3 0.62 0.05; visual box size=3 0.62 0.05
Joints:
- added joint fixed1: type fixed, parent base_link, child railing1, origin xyz=0 0.3 0.3 rpy=0 0 0, axis 0 0 1, limit lower=-2.6 upper=2.6 effort=1000 velocity=1000
- added joint fixed2: type fixed, parent base_link, child railing2, origin xyz=0 -0.3 0.3 rpy=0 0 0, axis 0 0 1, limit lower=-2.6 upper=2.6 effort=1000 velocity=1000
- added joint fixed3: type fixed, parent base_link, child railing3, origin xyz=0 0.0 0.25 rpy=0 0 0, axis 0 0 1, limit lower=-2.6 upper=2.6 effort=1000 velocity=1000

File: urdf/red_cylinder.urdf (robot description, URDF)
Before this commit: robot red_cylinder, 1 links, 0 joints
Links:
- link base_link: mass 0.00001 -> 0.14; geometry collision mesh filename=file:///home/saurabharora/catkin_ws/src/sawyer_irl_project/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; visual mesh filename=file:///home/saurabharora/catkin_ws/src/sawyer_irl_project/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
