Commit message: First push

File: urdf/OnionCenter.urdf (robot description, URDF)
Before this commit: robot blue_cylinder, 2 links, 1 joints
Links:
- link base_link: geometry collision mesh filename=file:///home/psuresh/catkin_ws/src/sawyer_irl_project/meshe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; visual mesh filename=file:///home/psuresh/catkin_ws/src/sawyer_irl_project/meshe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
- link film: geometry collision mesh filename=file:///home/psuresh/catkin_ws/src/sawyer_irl_project/meshe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; visual mesh filename=file:///home/psuresh/catkin_ws/src/sawyer_irl_project/meshe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

File: urdf/red_cylinder.urdf (robot description, URDF)
Before this commit: robot red_cylinder, 1 links, 0 joints
Links:
- link base_link: geometry collision mesh filename=file:///home/psuresh/catkin_ws/src/sawyer_irl_project/meshe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; visual mesh filename=file:///home/psuresh/catkin_ws/src/sawyer_irl_project/meshe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
