Commit message: Relative paths changed

File: urdf/Onion0.urdf (robot description, URDF)
Before this commit: robot blue_cylinder, 2 links, 1 joints
Links:
- link base_link: geometry collision mesh filename=package://sawyer_irl_project/meshes/custom_onion.STL; visual mesh filename=package://sawyer_irl_project/meshes/custom_onion.STL
- link film: geometry collision mesh filename=package://sawyer_irl_project/meshes/custom_onion_defect.STL; visual mesh filename=package://sawyer_irl_project/meshes/custom_onion_defect.STL

File: urdf/OnionCenter.urdf (robot description, URDF)
Before this commit: robot blue_cylinder, 2 links, 1 joints
Links:
- link base_link: geometry collision mesh filename=package://sawyer_irl_project/meshes/custom_onion.STL; visual mesh filename=package://sawyer_irl_project/meshes/custom_onion.STL
- link film: geometry collision mesh filename=package://sawyer_irl_project/meshes/custom_onion_defect.STL; visual mesh filename=package://sawyer_irl_project/meshes/custom_onion_defect.STL

File: urdf/red_cylinder.urdf (robot description, URDF)
Before this commit: robot red_cylinder, 1 links, 0 joints
Links:
- link base_link: geometry collision mesh filename=package://sawyer_irl_project/meshes/custom_onion.STL; visual mesh filename=package://sawyer_irl_project/meshes/custom_onion.STL
